File: HARDWARE/USB-GIGABIT-Rev.E/USB-GIGABIT_Rev_E.kicad_sch (KiCad schematic)
At the start: 52 parts, among them U2 NA(93LC46), U3 RTL8153VC-CG, U4 SY8089AAAC, X1 25MHz/20ppm/20pF/4P/3225

Commit message: Saved with Kicad 9.0
Parts:
- FB1: value 600OHM/2A/UPZ2012E-601-2R0TF/0805 -> 600OHM/2A/UPZ2012E-601-2R0TF/0805
